File: breadboardpower.brd (EAGLE design)
At the start: 33 x 52.1 mm, 11 parts, among them J1 DCJ0202, J2POS 571-0500, J3NEG 571-0500

Commit message: Add files via upload
Routing:
- net VCC: track 71.2 -> 83.3 mm
- net POS: track 82.1 -> 79.8 mm
- net HEAD: track 43.9 -> 42.8 mm
Other:
- board text added: "BreadBoardPower V4"
- board text removed: "BreadBoardPower V3"
Changed lines of the file:
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@@
 <?xml version="1.0" encoding="utf-8"?>
 <!DOCTYPE eagle SYSTEM "eagle.dtd">
-<eagle version="8.4.1">
+<eagle version="9.6.2">
 <drawing>
 <settings>
@@
 <setting verticaltext="up"/>
 </settings>
-<grid distance="0.1" unitdist="inch" unit="inch" style="lines" multiple="1" display="yes" altdistance="0.025" altunitdist="inch" altunit="inch"/>
+<grid distance="0.05" unitdist="inch" unit="inch" style="lines" multiple="1" display="yes" altdistance="0.025" altunitdist="inch" altunit="inch"/>
 <layers>
 <layer number="1" name="Top" color="4" fill="1" visible="yes" active="yes"/>
@@
 <wire x1="33.02" y1="2.54" x2="30.48" y2="0" width="0.1524" layer="20" curve="-90"/>
 <dimension x1="30.48" y1="49.53" x2="30.48" y2="2.54" x3="43.18" y3="26.035" textsize="1.778" layer="47" unit="inch"/>
-<text x="13.97" y="20.32" size="1.778" layer="26" rot="MR90">BreadBoardPower V3</text>
+<text x="13.97" y="20.32" size="1.778" layer="26" rot="MR90">BreadBoardPower V4</text>
 <text x="31.115" y="1.905" size="1.778" layer="25">+</text>
 <text x="31.115" y="46.355" size="1.778" layer="25">+</text>
@@
 </variantdefs>
 <classes>
-<class number="0" name="default" width="0" drill="0">
+<class number="0" name="default" width="1.016" drill="0">
 </class>
 </classes>
@@
 <param name="checkRestrict" value="1"/>
 <param name="checkStop" value="0"/>
+<param name="checkValues" value="0"/>
+<param name="checkNames" value="1"/>
+<param name="checkWireStubs" value="1"/>
+<param name="checkPolygonWidth" value="0"/>
 <param name="useDiameter" value="13"/>
 <param name="maxErrors" value="50"/>
@@
 <attribute name="VALUE" x="17.78" y="43.815" size="1.27" layer="27"/>
 </element>
-<element name="U$1" library="oshw" package="OSHW_5MM" value="" x="10.16" y="33.02" rot="MR90"/>
+<element name="U$1" library="oshw" package="OSHW_5MM" value="" x="10.16" y="33.02" smashed="yes" rot="MR90"/>
 </elements>
 <signals>
@@
 <contactref element="J1" pad="1"/>
 <contactref element="C1" pad="+"/>
-<wire x1="19.1008" y1="39.37" x2="6.096" y2="39.37" width="0.254" layer="16"/>
-<wire x1="6.096" y1="39.37" x2="3.81" y2="39.37" width="0.254" layer="16"/>
-<wire x1="21.59" y1="18.034" x2="21.59" y2="12.446" width="0.254" layer="16"/>
-<wire x1="21.59" y1="12.446" x2="21.5392" y2="12.2428" width="0.254" layer="16"/>
-<wire x1="21.59" y1="18.034" x2="21.5392" y2="18.2372" width="0.254" layer="16"/>
-<wire x1="11.43" y1="7.112" x2="3.302" y2="15.24" width="0.254" layer="16"/>
-<wire x1="11.938" y1="7.112" x2="11.43" y2="7.112" width="0.254" layer="16"/>
-<wire x1="11.938" y1="7.112" x2="11.99" y2="6.985" width="0.254" layer="16"/>
-<wire x1="21.082" y1="12.192" x2="21.336" y2="12.192" width="0.254" layer="1"/>
-<wire x1="16.51" y1="7.62" x2="21.082" y2="12.192" width="0.254" layer="1"/>
-<wire x1="12.7" y1="7.62" x2="16.51" y2="7.62" width="0.254" layer="1"/>
-<wire x1="12.192" y1="7.112" x2="12.7" y2="7.62" width="0.254" layer="1"/>
-<wire x1="21.336" y1="12.192" x2="21.5392" y2="12.2428" width="0.254" layer="1"/>
-<wire x1="12.192" y1="7.112" x2="11.99" y2="6.985" width="0.254" layer="1"/>
-<wire x1="6.096" y1="18.034" x2="6.096" y2="39.37" width="0.254" layer="16"/>
-<wire x1="3.302" y1="15.24" x2="6.096" y2="18.034" width="0.254" layer="16"/>
-<wire x1="3.302" y1="15.24" x2="2.54" y2="15.24" width="0.254" layer="16"/>
+<wire x1="2.54" y1="20.32" x2="2.54" y2="15.24" width="1.016" layer="16"/>
+<wire x1="6.985" y1="24.765" x2="2.54" y2="20.32" width="1.016" layer="16"/>
+<wire x1="6.985" y1="36.195" x2="6.985" y2="24.765" width="1.016" layer="16"/>
+<wire x1="3.81" y1="39.37" x2="6.985" y2="36.195" width="1.016" layer="16"/>
+<wire x1="21.59" y1="17.78" x2="21.59" y2="12.7" width="1.016" layer="16"/>
+<wire x1="21.59" y1="12.7" x2="21.5392" y2="12.2428" width="1.016" layer="16"/>
+<wire x1="21.59" y1="17.78" x2="21.5392" y2="18.2372" width="1.016" layer="16"/>
+<wire x1="15.875" y1="6.985" x2="11.99" y2="6.985" width="1.016" layer="16"/>
+<wire x1="20.955" y1="12.065" x2="15.875" y2="6.985" width="1.016" layer="16"/>
+<wire x1="20.955" y1="12.065" x2="21.5392" y2="12.2428" width="1.016" layer="16"/>
+<wire x1="19.685" y1="31.115" x2="19.685" y2="39.37" width="1.016" layer="16"/>
+<wire x1="22.225" y1="28.575" x2="19.685" y2="31.115" width="1.016" layer="16"/>
+<wire x1="22.225" y1="19.05" x2="22.225" y2="28.575" width="1.016" layer="16"/>
+<wire x1="21.59" y1="18.415" x2="22.225" y2="19.05" width="1.016" layer="16"/>
+<wire x1="19.685" y1="39.37" x2="19.1008" y2="39.37" width="1.016" layer="16"/>
+<wire x1="21.59" y1="18.415" x2="21.5392" y2="18.2372" width="1.016" layer="16"/>
+<wire x1="19.1008" y1="39.37" x2="3.81" y2="39.37" width="1.016" layer="1"/>
 </signal>
 <signal name="GND">
@@
 <contactref element="JP1" pad="7"/>
 <contactref element="JP1" pad="9"/>
-<wire x1="21.59" y1="2.54" x2="19.05" y2="2.54" width="0.254" layer="16"/>
-<wire x1="21.59" y1="2.54" x2="24.13" y2="2.54" width="0.254" layer="16"/>
-<wire x1="24.13" y1="2.54" x2="26.67" y2="2.54" width="0.254" layer="16"/>
-<wire x1="26.67" y1="2.54" x2="29.21" y2="2.54" width="0.254" layer="16"/>
-<wire x1="16.51" y1="18.034" x2="16.51" y2="15.24" width="0.254" layer="16"/>
-<wire x1="16.51" y1="15.24" x2="16.51" y2="12.446" width="0.254" layer="16"/>
-<wire x1="16.51" y1="12.446" x2="16.5608" y2="12.2428" width="0.254" layer="16"/>
-<wire x1="16.51" y1="18.034" x2="16.5608" y2="18.2372" width="0.254" layer="16"/>
-<wire x1="16.51" y1="15.24" x2="10.795" y2="15.24" width="0.254" layer="16"/>
-<wire x1="29.718" y1="48.26" x2="16.51" y2="48.26" width="0.254" layer="16"/>
-<wire x1="30.48" y1="47.498" x2="29.718" y2="48.26" width="0.254" layer="16"/>
-<wire x1="30.48" y1="44.196" x2="30.48" y2="47.498" width="0.254" layer="16"/>
-<wire x1="16.764" y1="30.48" x2="30.48" y2="44.196" width="0.254" layer="16"/>
-<wire x1="16.764" y1="18.288" x2="16.764" y2="30.48" width="0.254" layer="16"/>
-<wire x1="16.764" y1="18.288" x2="16.5608" y2="18.2372" width="0.254" layer="16"/>
-<wire x1="19.05" y1="3.302" x2="19.05" y2="2.54" width="0.254" layer="16"/>
-<wire x1="16.764" y1="5.588" x2="19.05" y2="3.302" width="0.254" layer="16"/>
-<wire x1="16.764" y1="12.192" x2="16.764" y2="5.588" width="0.254" layer="16"/>
-<wire x1="16.764" y1="12.192" x2="16.5608" y2="12.2428" width="0.254" layer="16"/>
+<wire x1="21.59" y1="2.54" x2="19.05" y2="2.54" width="1.016" layer="16"/>
+<wire x1="21.59" y1="2.54" x2="24.13" y2="2.54" width="1.016" layer="16"/>
+<wire x1="24.13" y1="2.54" x2="26.67" y2="2.54" width="1.016" layer="16"/>
+<wire x1="26.67" y1="2.54" x2="29.21" y2="2.54" width="1.016" layer="16"/>
+<wire x1="16.51" y1="17.78" x2="16.51" y2="15.24" width="1.016" layer="16"/>
+<wire x1="16.51" y1="15.24" x2="16.51" y2="12.7" width="1.016" layer="16"/>
+<wire x1="16.51" y1="12.7" x2="16.5608" y2="12.2428" width="1.016" layer="16"/>
+<wire x1="16.51" y1="17.78" x2="16.5608" y2="18.2372" width="1.016" layer="16"/>
+<wire x1="16.51" y1="15.24" x2="10.795" y2="15.24" width="1.016" layer="16"/>
+<wire x1="16.51" y1="46.355" x2="16.51" y2="48.26" width="1.016" layer="16"/>
+<wire x1="8.255" y1="38.1" x2="16.51" y2="46.355" width="1.016" layer="16"/>
+<wire x1="8.255" y1="17.145" x2="8.255" y2="38.1" width="1.016" layer="16"/>
+<wire x1="10.16" y1="15.24" x2="8.255" y2="17.145" width="1.016" layer="16"/>
+<wire x1="12.7" y1="2.54" x2="19.05" y2="2.54" width="1.016" layer="16"/>
+<wire x1="10.16" y1="5.08" x2="12.7" y2="2.54" width="1.016" layer="16"/>
+<wire x1="10.16" y1="15.24" x2="10.16" y2="5.08" width="1.016" layer="16"/>
+<wire x1="10.16" y1="15.24" x2="10.795" y2="15.24" width="1.016" layer="16"/>
 </signal>
 <signal name="N$2">
 <contactref element="LED1" pad="A"/>
 <contactref element="R1" pad="2"/>
-<wire x1="6.35" y1="48.26" x2="4.445" y2="48.26" width="0.254" layer="1"/>
+<wire x1="6.35" y1="48.26" x2="4.445" y2="48.26" width="1.016" layer="16"/>
 </signal>
 <signal name="HEAD">
@@
 <contactref element="JP3" pad="7"/>
 <contactref element="JP3" pad="9"/>
-<wire x1="10.922" y1="26.67" x2="10.922" y2="17.78" width="0.254" layer="16"/>
-<wire x1="21.59" y1="37.338" x2="10.922" y2="26.67" width="0.254" layer="16"/>
-<wire x1="21.59" y1="46.99" x2="21.59" y2="37.338" width="0.254" layer="16"/>
-<wire x1="10.922" y1="17.78" x2="10.795" y2="17.78" width="0.254" layer="16"/>
-<wire x1="21.59" y1="46.99" x2="19.05" y2="46.99" width="0.254" layer="16"/>
-<wire x1="21.59" y1="46.99" x2="24.13" y2="46.99" width="0.254" layer="16"/>
-<wire x1="24.13" y1="46.99" x2="26.67" y2="46.99" width="0.254" layer="16"/>
-<wire x1="26.67" y1="46.99" x2="29.21" y2="46.99" width="0.254" layer="16"/>
+<wire x1="10.795" y1="38.735" x2="10.795" y2="17.78" width="1.016" layer="16"/>
+<wire x1="19.05" y1="46.99" x2="10.795" y2="38.735" width="1.016" layer="16"/>
+<wire x1="19.05" y1="46.99" x2="21.59" y2="46.99" width="1.016" layer="16"/>
+<wire x1="21.59" y1="46.99" x2="24.13" y2="46.99" width="1.016" layer="16"/>
+<wire x1="24.13" y1="46.99" x2="26.67" y2="46.99" width="1.016" layer="16"/>
+<wire x1="26.67" y1="46.99" x2="29.21" y2="46.99" width="1.016" layer="16"/>
 </signal>
 </signals>
-<errors>
-</errors>
+<mfgpreviewcolors>
+<mfgpreviewcolor name="soldermaskcolor" color="0xC8008000"/>
+<mfgpreviewcolor name="silkscreencolor" color="0xFFFEFEFE"/>
+<mfgpreviewcolor name="backgroundcolor" color="0xFF282828"/>
+<mfgpreviewcolor name="coppercolor" color="0xFFFFBF00"/>
+<mfgpreviewcolor name="substratecolor" color="0xFF786E46"/>
+</mfgpreviewcolors>
 </board>
 </drawing>
